Commit message: slam mode ready in ROS

File: realsense-ros-2.3.2/realsense2_description/urdf/test_d435_camera.urdf.xacro (robot description, xacro)
@@ -9,3 +9,7 @@
     <origin xyz="0 0 0" rpy="0 0 0"/>
   </xacro:sensor_d435>
+<!--  <link name="d435i_link" />-->
+<!--  <xacro:sensor_d435 parent="d435i_link" use_nominal_extrinsics="$(arg use_nominal_extrinsics)" add_plug="$(arg add_plug)" use_mesh="$(arg use_mesh)">-->
+<!--    <origin xyz="0 0 0" rpy="0 0 0"/>-->
+<!--  </xacro:sensor_d435>-->
 </robot>

Commit message: updated slam mode details, started localization

File: realsense-ros-2.3.2/realsense2_description/urdf/test_d435_camera.urdf.xacro (robot description, xacro)
@@ -9,7 +9,3 @@
     <origin xyz="0 0 0" rpy="0 0 0"/>
   </xacro:sensor_d435>
-<!--  <link name="d435i_link" />-->
-<!--  <xacro:sensor_d435 parent="d435i_link" use_nominal_extrinsics="$(arg use_nominal_extrinsics)" add_plug="$(arg add_plug)" use_mesh="$(arg use_mesh)">-->
-<!--    <origin xyz="0 0 0" rpy="0 0 0"/>-->
-<!--  </xacro:sensor_d435>-->
 </robot>
